Commit message: add package robin_maze_solver

File: src/robin_description/urdf/common_properties.xacro (robot description, xacro)
@@ -1,3 +1,3 @@
-<!-- <?xml version="1.0"?> -->
+<?xml version="1.0"?>
 <robot xmlns:xacro="http://www.ros.org/wiki/xacro">
     <material name="blue">

File: src/robin_description/urdf/mobile_base.xacro (robot description, xacro)
@@ -1,42 +1,9 @@
-<robot xmlns:xacro="http://www.ros.org/wiki/xacro" name="robin">
-    <!-- ===================== MACRO INERTIA ===================== -->
-    <xacro:macro name="box_inertia" params="m x y z o_xyz o_rpy">
-        <inertial>
-            <mass value="${m}"/>
-            <origin xyz="${o_xyz}" rpy="${o_rpy}"/>
-            <inertia
-                ixx="${m*(y*y+z*z)/12.0}" ixy="0" ixz="0"
-                iyy="${m*(x*x+z*z)/12.0}" iyz="0"
-                izz="${m*(x*x+y*y)/12.0}"/>
-        </inertial>
-    </xacro:macro>
-    <xacro:macro name="cylinder_inertia" params="m r l o_xyz o_rpy">
-        <inertial>
-            <mass value="${m}"/>
-            <origin xyz="${o_xyz}" rpy="${o_rpy}"/>
-            <inertia
-                ixx="${m*(3*r*r+l*l)/12.0}" ixy="0" ixz="0"
-                iyy="${m*(3*r*r+l*l)/12.0}" iyz="0"
-                izz="${m*r*r/2.0}"/>
-        </inertial>
-    </xacro:macro>
-    <xacro:macro name="sphere_inertia" params="m r o_xyz o_rpy">
-        <inertial>
-            <mass value="${m}"/>
-            <origin xyz="${o_xyz}" rpy="${o_rpy}"/>
-            <inertia
-                ixx="${2.0*m*r*r/5.0}" ixy="0" ixz="0"
-                iyy="${2.0*m*r*r/5.0}" iyz="0"
-                izz="${2.0*m*r*r/5.0}"/>
-        </inertial>
-    </xacro:macro>
-    <!-- ===================== PROPERTIES ===================== -->
-    <xacro:property name="base_length" value="0.6" />
-    <xacro:property name="base_width"  value="0.4" />
-    <xacro:property name="base_height" value="0.2" />
-    <xacro:property name="wheel_radius" value="0.1" />
-    <xacro:property name="wheel_length" value="0.05" />
-    <xacro:property name="wheel_separation" value="${base_width + wheel_length}" />
-    <!-- ===================== BASE ===================== -->
+<?xml version="1.0"?>
+<robot xmlns:xacro="http://www.ros.org/wiki/xacro">
+    <xacro:property name="base_length" value="0.15" />
+    <xacro:property name="base_width" value="0.15" />
+    <xacro:property name="base_height" value="0.05" />
+    <xacro:property name="wheel_radius" value="0.03" />
+    <xacro:property name="wheel_length" value="0.02" />
     <link name="base_footprint" />
     <link name="base_link">
@@ -46,7 +13,5 @@
             </geometry>
             <origin xyz="0 0 ${base_height / 2.0}" rpy="0 0 0" />
-            <material name="blue">
-                <color rgba="0.2 0.2 0.8 1.0"/>
-            </material>
+            <material name="blue" />
         </visual>
         <collision>
@@ -57,7 +22,6 @@
         </collision>
         <xacro:box_inertia m="5.0" x="${base_length}" y="${base_width}" z="${base_height}"
-                            o_xyz="0 0 ${base_height / 2.0}" o_rpy="0 0 0" />
+                           o_xyz="0 0 ${base_height / 2.0}" o_rpy="0 0 0" />
     </link>
-    <!-- ===================== WHEEL MACRO ===================== -->
     <xacro:macro name="wheel_link" params="prefix">
         <link name="${prefix}_wheel_link">
@@ -67,7 +31,5 @@
                 </geometry>
                 <origin xyz="0 0 0" rpy="${pi / 2.0} 0 0" />
-                <material name="grey">
-                    <color rgba="0.4 0.4 0.4 1.0"/>
-                </material>
+                <material name="grey" />
             </visual>
             <collision>
@@ -83,6 +45,5 @@
     <xacro:wheel_link prefix="right" />
     <xacro:wheel_link prefix="left" />
-    <!-- ===================== CASTER ===================== -->
-    <link name="caster_wheel_link">
+    <link name="caster_front_wheel_link">
         <visual>
             <geometry>
@@ -90,7 +51,5 @@
             </geometry>
             <origin xyz="0 0 0" rpy="0 0 0" />
-            <material name="grey">
-                <color rgba="0.4 0.4 0.4 1.0"/>
-            </material>
+            <material name="grey" />
         </visual>
         <collision>
@@ -101,30 +60,49 @@
         </collision>
         <xacro:sphere_inertia m="0.5" r="${wheel_radius / 2.0}"
-                                o_xyz="0 0 0" o_rpy="0 0 0" />
+                              o_xyz="0 0 0" o_rpy="0 0 0" />
     </link>
-    <!-- ===================== JOINTS ===================== -->
+    <link name="caster_rear_wheel_link">
+        <visual>
+            <geometry>
+                <sphere radius="${wheel_radius / 2.0}" />
+            </geometry>
+            <origin xyz="0 0 0" rpy="0 0 0" />
+            <material name="grey" />
+        </visual>
+        <collision>
+            <geometry>
+                <sphere radius="${wheel_radius / 2.0}" />
+            </geometry>
+            <origin xyz="0 0 0" rpy="0 0 0" />
+        </collision>
+        <xacro:sphere_inertia m="0.5" r="${wheel_radius / 2.0}"
+                              o_xyz="0 0 0" o_rpy="0 0 0" />
+    </link>
     <joint name="base_joint" type="fixed">
         <parent link="base_footprint" />
-        <child  link="base_link" />
+        <child link="base_link" />
         <origin xyz="0 0 ${wheel_radius}" rpy="0 0 0"/>
     </joint>
     <joint name="base_right_wheel_joint" type="continuous">
         <parent link="base_link" />
-        <child  link="right_wheel_link" />
-        <origin xyz="${-base_length / 4.0} ${-(base_width + wheel_length) / 2.0} 0" rpy="0 0 0" />
+        <child link="right_wheel_link" />
+        <origin xyz="${-base_length*0.0 / 4.0} ${-(base_width + wheel_length) / 2.0} 0" rpy="0 0 0" />
         <axis xyz="0 1 0" />
-        <limit effort="100.0" velocity="100.0" />
     </joint>
     <joint name="base_left_wheel_joint" type="continuous">
         <parent link="base_link" />
-        <child  link="left_wheel_link" />
-        <origin xyz="${-base_length / 4.0} ${(base_width + wheel_length) / 2.0} 0" rpy="0 0 0" />
+        <child link="left_wheel_link" />
+        <origin xyz="${-base_length*0.0 / 4.0} ${(base_width + wheel_length) / 2.0} 0" rpy="0 0 0" />
         <axis xyz="0 1 0" />
-        <limit effort="100.0" velocity="100.0" />
     </joint>
-    <joint name="base_caster_wheel_joint" type="fixed">
+    <joint name="base_caster_front_wheel_joint" type="fixed">
         <parent link="base_link" />
-        <child  link="caster_wheel_link" />
+        <child link="caster_front_wheel_link" />
         <origin xyz="${base_length / 3.0} 0 ${-wheel_radius / 2.0}" rpy="0 0 0" />
     </joint>
+    <joint name="base_caster_rear_wheel_joint" type="fixed">
+        <parent link="base_link" />
+        <child link="caster_rear_wheel_link" />
+        <origin xyz="${-base_length / 3.0} 0 ${-wheel_radius / 2.0}" rpy="0 0 0" />
+    </joint>
 </robot>

File: src/robin_description/urdf/mobile_base_gazebo.xacro (robot description, xacro)
@@ -1,56 +1,31 @@
+<?xml version="1.0"?>
 <robot xmlns:xacro="http://www.ros.org/wiki/xacro">
-    <gazebo reference="caster_wheel_link">
+    <gazebo reference="caster_front_wheel_link">
         <mu1 value="0.1" />
         <mu2 value="0.1" />
     </gazebo>
-    <gazebo reference="left_wheel_link">
-        <mu1 value="1.0" />
-        <mu2 value="1.0" />
-    </gazebo>
-    <gazebo reference="right_wheel_link">
-        <mu1 value="1.0" />
-        <mu2 value="1.0" />
+    <gazebo reference="caster_rear_wheel_link">
+        <mu1 value="0.1" />
+        <mu2 value="0.1" />
     </gazebo>
     <gazebo>
-        <plugin filename="gz-sim-joint-controller-system"
-                name="gz::sim::systems::JointController">
-            <joint_name>base_left_wheel_joint</joint_name>
-            <initial_velocity>0.0</initial_velocity>
+        <plugin
+            filename="gz-sim-diff-drive-system"
+            name="gz::sim::systems::DiffDrive">
+            <left_joint>base_left_wheel_joint</left_joint>
+            <right_joint>base_right_wheel_joint</right_joint>
+            <wheel_separation>0.45</wheel_separation>
+            <wheel_radius>0.1</wheel_radius>
+            <frame_id>odom</frame_id>
+            <child_frame_id>base_footprint</child_frame_id>
         </plugin>
     </gazebo>
     <gazebo>
-        <plugin filename="gz-sim-joint-controller-system"
-                name="gz::sim::systems::JointController">
-            <joint_name>base_right_wheel_joint</joint_name>
-            <initial_velocity>0.0</initial_velocity>
-        </plugin>
-    </gazebo>
-    <gazebo>
-        <plugin filename="gz-sim-joint-state-publisher-system"
-                name="gz::sim::systems::JointStatePublisher">
-            <topic>joint_state</topic>
+        <plugin
+            filename="gz-sim-joint-state-publisher-system"
+            name="gz::sim::systems::JointStatePublisher">
             <joint_name>base_left_wheel_joint</joint_name>
             <joint_name>base_right_wheel_joint</joint_name>
         </plugin>
     </gazebo>
-    <gazebo>
-        <plugin filename="gz-sim-pose-publisher-system"
-                name="gz::sim::systems::PosePublisher">
-            <publish_link_pose>true</publish_link_pose>
-            <publish_visual_pose>true</publish_visual_pose>
-            <publish_collision_pose>false</publish_collision_pose>
-            <publish_nested_model_pose>true</publish_nested_model_pose>
-            <use_pose_vector_msg>true</use_pose_vector_msg>
-            <update_frequency>30</update_frequency>
-        </plugin>
-    </gazebo>
-    <gazebo>
-        <plugin filename="gz-sim-odometry-publisher-system"
-                name="gz::sim::systems::OdometryPublisher">
-            <odom_frame>odom</odom_frame>
-            <robot_base_frame>base_footprint</robot_base_frame>
-            <odom_publish_frequency>30</odom_publish_frequency>
-            <dimensions>2</dimensions>
-        </plugin>
-    </gazebo>
 </robot>
